Commit message: more stuf

File: description/robot_core.xacro (robot description, xacro)
@@ -68,5 +68,5 @@
 </link>
 <gazebo reference="left_wheel">
-    <material>Gazebo/blue</material>
+    <material>Gazebo/Blue</material>
 </gazebo>
 <!-- RIGHT WHEEL LINK -->
@@ -120,4 +120,6 @@
 <gazebo reference="caster_wheel">
     <material>Gazebo/Black</material>
+    <mu1 value="0.001"/>
+    <mu2 value="0.001"/>
 </gazebo>
 </robot>

Commit message: update code

File: description/robot_core.xacro (robot description, xacro)
@@ -19,4 +19,12 @@
 <!-- BASE LINK -->
 <link name="base_link" >
+</link>
+ <!-- BASE_FOOTPRINT LINK -->
+ <joint name="base_footprint_joint" type="fixed">
+    <parent link="base_link"/>
+    <child link="base_footprint"/>
+    <origin xyz="0 0 0" rpy="0 0 0"/>
+</joint>
+<link name="base_footprint">
 </link>
 <!-- CHASSIS LINK -->
